File: hardware/kicad/ESP32-P4 Display Development Daughterboard.kicad_sch (KiCad schematic)
At the start: 0 parts

Commit message: hardware: complete Phase 2 schematic capture
Other:
- added sheet 240 mA Backlight (09_backlight.kicad_sch)
- added sheet Bench 24 V Input (01_bench_input.kicad_sch)
- added sheet Display Rails and Sequencing (06_display_power_sequence.kicad_sch)
- added sheet GT9271 Touch Interface (08_touch.kicad_sch)
- added sheet LM5176 Vehicle Buck-Boost (03_vehicle_buckboost.kicad_sch)
- added sheet MIPI DSI and LCD Connector (07_mipi_panel.kicad_sch)
- added sheet Nano Headers and Debug (10_headers_debug.kicad_sch)
- added sheet Source ORing (04_source_oring.kicad_sch)
- added sheet System 5 V and Nano Feed (05_system_5v.kicad_sch)
- added sheet Vehicle Input Protection (02_vehicle_protection.kicad_sch)
- note added: "PHASE 2 SCHEMATIC — PCB layout not started. Read docs/design-notes/schematic-calculations.md and schematic-review.md before review."
- company: (none) -> sydude/ESP32-P4-Display-Development-Daughterboard
- title: (none) -> ESP32-P4 Displayman Development Daughterboard
Changed lines of the file:
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@@
-(kicad_sch
-	(version 20260306)
-	(generator "eeschema")
-	(generator_version "10.0")
-	(paper "A4")
-	(sheet_instances
-		(path "/"
-			(page "1")
-		)
-	)
-	(embedded_fonts no)
+(kicad_sch (version 20230121) (generator eeschema)
+  (paper "A3")
+  (title_block (title "ESP32-P4 Displayman Development Daughterboard") (date "2026-09-16") (rev "Phase 2 / v0.1") (company "sydude/ESP32-P4-Display-Development-Daughterboard"))
+  (text "PHASE 2 SCHEMATIC — PCB layout not started. Read docs/design-notes/schematic-calculations.md and schematic-review.md before review." (at 20 20 0) (effects (font (size 1.8 1.8)) (justify left bottom)))
+  (sheet (at 25 35) (size 105 40) (stroke (width 0) (type solid)) (fill (color 0 0 0 0.0000))
+    (property "Sheetname" "Bench 24 V Input" (at 25 34.2 0) (effects (font (size 1.27 1.27)) (justify left bottom)))
+    (property "Sheetfile" "01_bench_input.kicad_sch" (at 25 75.8 0) (effects (font (size 1.0 1.0)) (justify left top)))
+    (instances (project "ESP32-P4 Display Development Daughterboard" (path "/ee8cb40b-4ed6-449e-895a-459b7616a52d" (page "2"))))
+  )
+  (sheet (at 150 35) (size 105 40) (stroke (width 0) (type solid)) (fill (color 0 0 0 0.0000))
+    (property "Sheetname" "Vehicle Input Protection" (at 150 34.2 0) (effects (font (size 1.27 1.27)) (justify left bottom)))
+    (property "Sheetfile" "02_vehicle_protection.kicad_sch" (at 150 75.8 0) (effects (font (size 1.0 1.0)) (justify left top)))
+    (instances (project "ESP32-P4 Display Development Daughterboard" (path "/ee8cb40b-4ed6-449e-895a-459b7616a52d" (page "3"))))
+  )
+  (sheet (at 275 35) (size 105 40) (stroke (width 0) (type solid)) (fill (color 0 0 0 0.0000))
+    (property "Sheetname" "LM5176 Vehicle Buck-Boost" (at 275 34.2 0) (effects (font (size 1.27 1.27)) (justify left bottom)))
+    (property "Sheetfile" "03_vehicle_buckboost.kicad_sch" (at 275 75.8 0) (effects (font (size 1.0 1.0)) (justify left top)))
+    (instances (project "ESP32-P4 Display Development Daughterboard" (path "/ee8cb40b-4ed6-449e-895a-459b7616a52d" (page "4"))))
+  )
+  (sheet (at 25 90) (size 105 40) (stroke (width 0) (type solid)) (fill (color 0 0 0 0.0000))
+    (property "Sheetname" "Source ORing" (at 25 89.2 0) (effects (font (size 1.27 1.27)) (justify left bottom)))
+    (property "Sheetfile" "04_source_oring.kicad_sch" (at 25 130.8 0) (effects (font (size 1.0 1.0)) (justify left top)))
+    (instances (project "ESP32-P4 Display Development Daughterboard" (path "/ee8cb40b-4ed6-449e-895a-459b7616a52d" (page "5"))))
+  )
+  (sheet (at 150 90) (size 105 40) (stroke (width 0) (type solid)) (fill (color 0 0 0 0.0000))
+    (property "Sheetname" "System 5 V and Nano Feed" (at 150 89.2 0) (effects (font (size 1.27 1.27)) (justify left bottom)))
+    (property "Sheetfile" "05_system_5v.kicad_sch" (at 150 130.8 0) (effects (font (size 1.0 1.0)) (justify left top)))
+    (instances (project "ESP32-P4 Display Development Daughterboard" (path "/ee8cb40b-4ed6-449e-895a-459b7616a52d" (page "6"))))
+  )
+  (sheet (at 275 90) (size 105 40) (stroke (width 0) (type solid)) (fill (color 0 0 0 0.0000))
+    (property "Sheetname" "Display Rails and Sequencing" (at 275 89.2 0) (effects (font (size 1.27 1.27)) (justify left bottom)))
+    (property "Sheetfile" "06_display_power_sequence.kicad_sch" (at 275 130.8 0) (effects (font (size 1.0 1.0)) (justify left top)))
+    (instances (project "ESP32-P4 Display Development Daughterboard" (path "/ee8cb40b-4ed6-449e-895a-459b7616a52d" (page "7"))))
+  )
+  (sheet (at 25 145) (size 105 40) (stroke (width 0) (type solid)) (fill (color 0 0 0 0.0000))
+    (property "Sheetname" "MIPI DSI and LCD Connector" (at 25 144.2 0) (effects (font (size 1.27 1.27)) (justify left bottom)))
+    (property "Sheetfile" "07_mipi_panel.kicad_sch" (at 25 185.8 0) (effects (font (size 1.0 1.0)) (justify left top)))
+    (instances (project "ESP32-P4 Display Development Daughterboard" (path "/ee8cb40b-4ed6-449e-895a-459b7616a52d" (page "8"))))
+  )
+  (sheet (at 150 145) (size 105 40) (stroke (width 0) (type solid)) (fill (color 0 0 0 0.0000))
+    (property "Sheetname" "GT9271 Touch Interface" (at 150 144.2 0) (effects (font (size 1.27 1.27)) (justify left bottom)))
+    (property "Sheetfile" "08_touch.kicad_sch" (at 150 185.8 0) (effects (font (size 1.0 1.0)) (justify left top)))
+    (instances (project "ESP32-P4 Display Development Daughterboard" (path "/ee8cb40b-4ed6-449e-895a-459b7616a52d" (page "9"))))
+  )
+  (sheet (at 275 145) (size 105 40) (stroke (width 0) (type solid)) (fill (color 0 0 0 0.0000))
+    (property "Sheetname" "240 mA Backlight" (at 275 144.2 0) (effects (font (size 1.27 1.27)) (justify left bottom)))
+    (property "Sheetfile" "09_backlight.kicad_sch" (at 275 185.8 0) (effects (font (size 1.0 1.0)) (justify left top)))
+    (instances (project "ESP32-P4 Display Development Daughterboard" (path "/ee8cb40b-4ed6-449e-895a-459b7616a52d" (page "10"))))
+  )
+  (sheet (at 25 200) (size 105 40) (stroke (width 0) (type solid)) (fill (color 0 0 0 0.0000))
+    (property "Sheetname" "Nano Headers and Debug" (at 25 199.2 0) (effects (font (size 1.27 1.27)) (justify left bottom)))
+    (property "Sheetfile" "10_headers_debug.kicad_sch" (at 25 240.8 0) (effects (font (size 1.0 1.0)) (justify left top)))
+    (instances (project "ESP32-P4 Display Development Daughterboard" (path "/ee8cb40b-4ed6-449e-895a-459b7616a52d" (page "11"))))
+  )
+  (sheet_instances (path "/" (page "1")))
 )
