File: hardware/kicad/ESP32-P4 Display Development Daughterboard.kicad_sch (KiCad schematic)
At the start: 0 parts

Commit message: Major fixes. Needs simplification, component organization and routing
Parts:
- added C201: 100nF 100V, Capacitor_SMD:C_0603_1608Metric, symbol Phase2:C201_100nF_100V
- added C202: 22uF 50V X7R, Capacitor_SMD:C_1210_3225Metric, symbol Phase2:C202_22uF_50V_X7R
- added C203: 100uF 50V, Capacitor_SMD:CP_Elec_10x10, symbol Phase2:C203_100uF_50V
- added C204: 10uF 50V, Capacitor_SMD:C_1210_3225Metric, symbol Phase2:C204_10uF_50V
- added C205: 100nF 100V, Capacitor_SMD:C_0603_1608Metric, symbol Phase2:C205_100nF_100V
- added C206: 100nF 100V, Capacitor_SMD:C_0603_1608Metric, symbol Phase2:C206_100nF_100V
- added C207: 82nF 25V X7R, Capacitor_SMD:C_0603_1608Metric, symbol Phase2:C304_82nF_X7R
- added C301: 47pF C0G, Capacitor_SMD:C_0402_1005Metric, symbol Phase2:C301_47pF_C0G
- added C302: 270pF C0G, Capacitor_SMD:C_0603_1608Metric, symbol Phase2:C302_270pF_C0G
- added C303: 100nF, Capacitor_SMD:C_0603_1608Metric, symbol Phase2:C303_100nF
- added C304: 82nF X7R, Capacitor_SMD:C_0603_1608Metric, symbol Phase2:C304_82nF_X7R
- added C305: 270pF C0G, Capacitor_SMD:C_0603_1608Metric, symbol Phase2:C305_270pF_C0G
- added C306: 1uF 16V, Capacitor_SMD:C_0603_1608Metric, symbol Phase2:C306_1uF_16V
- added C307: 100nF, Capacitor_SMD:C_0603_1608Metric, symbol Phase2:C307_100nF
- added C308: 100nF, Capacitor_SMD:C_0603_1608Metric, symbol Phase2:C308_100nF
- added C309: 220uF 35V, Capacitor_SMD:CP_Elec_10x12.5, symbol Phase2:C309_220uF_35V
- added C310: 22uF 50V, Capacitor_SMD:C_1210_3225Metric, symbol Phase2:C310_22uF_50V
- added C311: 220uF 35V, Capacitor_SMD:CP_Elec_10x12.5, symbol Phase2:C311_220uF_35V
- added C312: 22uF 50V, Capacitor_SMD:C_1210_3225Metric, symbol Phase2:C312_22uF_50V
- added C313: 22uF 50V, Capacitor_SMD:C_1210_3225Metric, symbol Phase2:C313_22uF_50V
- added C501: 470nF, Capacitor_SMD:C_0603_1608Metric, symbol Phase2:C501_470nF
- added C502: 2.2uF 10V, Capacitor_SMD:C_0603_1608Metric, symbol Phase2:C502_2.2uF_10V
- added C503: 1uF 10V, Capacitor_SMD:C_0603_1608Metric, symbol Phase2:C503_1uF_10V
- added C504: 22nF, Capacitor_SMD:C_0603_1608Metric, symbol Phase2:C504_22nF
- added C505: 4.7uF 100V, Capacitor_SMD:C_1210_3225Metric, symbol Phase2:C505_4.7uF_100V
- added C506: 4.7uF 100V, Capacitor_SMD:C_1210_3225Metric, symbol Phase2:C506_4.7uF_100V
- added C507: 47nF 100V, Capacitor_SMD:C_0603_1608Metric, symbol Phase2:C507_47nF_100V
- added C508: 22uF 10V, Capacitor_SMD:C_1210_3225Metric, symbol Phase2:C508_22uF_10V
- added C509: 22uF 10V, Capacitor_SMD:C_1210_3225Metric, symbol Phase2:C509_22uF_10V
- added C510: 22uF 10V, Capacitor_SMD:C_1210_3225Metric, symbol Phase2:C510_22uF_10V
- added C511: 22uF 10V, Capacitor_SMD:C_1210_3225Metric, symbol Phase2:C511_22uF_10V
- added C512: 10nF, Capacitor_SMD:C_0603_1608Metric, symbol Phase2:C512_10nF
- added C513: 1uF 10V, Capacitor_SMD:C_0603_1608Metric, symbol Phase2:C513_1uF_10V
- added C514: 1uF 10V, Capacitor_SMD:C_0603_1608Metric, symbol Phase2:C514_1uF_10V
- added C601: 6800uF 10V, Capacitor_THT:CP_Radial_D16.0mm_P7.50mm, symbol Phase2:C601_6800uF_10V
- added C602: 100pF C0G, Capacitor_SMD:C_0603_1608Metric, symbol Phase2:C602_100pF_C0G
- added C603: 1uF 10V, Capacitor_SMD:C_0603_1608Metric, symbol Phase2:C603_1uF_10V
- added C604: 2.2uF 6.3V, Capacitor_SMD:C_0603_1608Metric, symbol Phase2:C604_2.2uF_6.3V
- added C605: 2.2uF 6.3V, Capacitor_SMD:C_0603_1608Metric, symbol Phase2:C605_2.2uF_6.3V
- added C606: 4.7uF 6.3V, Capacitor_SMD:C_0603_1608Metric, symbol Phase2:C606_4.7uF_6.3V
- added C607: 1nF 50V C0G, Capacitor_SMD:C_0603_1608Metric, symbol Phase2:C602_100pF_C0G
- added C801: 1uF 10V, Capacitor_SMD:C_0603_1608Metric, symbol Phase2:C801_1uF_10V
- added C802: 4.7uF 6.3V, Capacitor_SMD:C_0603_1608Metric, symbol Phase2:C802_4.7uF_6.3V
- added C803: 100nF, Capacitor_SMD:C_0603_1608Metric, symbol Phase2:C803_100nF
- added C901: 10uF 50V, Capacitor_SMD:C_1210_3225Metric, symbol Phase2:C901_10uF_50V
- added C902: 100nF 100V, Capacitor_SMD:C_0603_1608Metric, symbol Phase2:C902_100nF_100V
- added C903: 1uF 10V, Capacitor_SMD:C_0603_1608Metric, symbol Phase2:C903_1uF_10V
- added C904: 1nF 50V, Capacitor_SMD:C_0603_1608Metric, symbol Phase2:C904_1nF_50V
- added C905: 2.2uF 50V, Capacitor_SMD:C_1210_3225Metric, symbol Phase2:C905_2.2uF_50V
- added C906: 1nF, Capacitor_SMD:C_0603_1608Metric, symbol Phase2:C906_1nF
- added C907: 1nF, Capacitor_SMD:C_0603_1608Metric, symbol Phase2:C907_1nF
- added C908: 10uF 50V, Capacitor_SMD:C_1210_3225Metric, symbol Phase2:C908_10uF_50V
- added D1001: GREEN, LED_SMD:LED_0603_1608Metric, symbol Phase2:D1001_GREEN
- added D1002: GREEN, LED_SMD:LED_0603_1608Metric, symbol Phase2:D1002_GREEN
- added D201: SM8S24CA-Q, Phase2:Bourns_DO-218AB, symbol Phase2:D201_SM8S24CA-Q
- added D301: BAT46W-E3-08, Diode_SMD:D_SOD-123, symbol Phase2:D301_BAT46W-E3-08
- added D302: BAT46W-E3-08, Diode_SMD:D_SOD-123, symbol Phase2:D302_BAT46W-E3-08
- added D601: SS34-E3/57T, Diode_SMD:D_SMA, symbol Phase2:D601_SS34-E3_57T
- added D602: 1N4148W, Diode_SMD:D_SOD-123, symbol Phase2:D602_1N4148W
- added D901: SS2H10-E3/52T, Diode_SMD:D_SMA, symbol Phase2:D901_SS2H10-E3_52T
- added F201: 5A TIME DELAY, Fuse:Fuseholder_Blade_Mini_Keystone_3568, symbol Phase2:F201_5A_TIME_DELAY
- added FB901: 600R@100MHz 1A, Inductor_SMD:L_0603_1608Metric, symbol Phase2:FB901_600R@100MHz_1A
- added J1001: SSQ-113-01-G-D, Phase2:Samtec_SSQ-113-01-G-D_BottomMount, symbol Phase2:J1001_NANO_P1_2x13
- added J1002: SSQ-113-01-G-D, Phase2:Samtec_SSQ-113-01-G-D_BottomMount, symbol Phase2:J1002_NANO_P2_2x13
- added J1003: DEBUG HEADER, Connector_PinHeader_2.54mm:PinHeader_2x05_P2.54mm_Vertical, symbol Phase2:J1003_DEBUG_HEADER
- added J201: VEHICLE 12V, Phase2:CONN_SD-43045-007_02_MOL, symbol Phase2:J201_VEHICLE_12V
- added J501: SERVICE LINK 5V, Jumper:SolderJumper-2_P1.3mm_Bridged_RoundedPad1.0x1.5mm, symbol Phase2:J501_SERVICE_LINK_5V
- added J701: NANO DSI 15P, Phase2:Amphenol_CON15_1X15_DRB_SFW_FCI, symbol Phase2:J701_NANO_DSI_15P
- added J702: DISPLAYMAN LCD 40P, Phase2:Molex_CON_5051104096, symbol Phase2:J702_DISPLAYMAN_LCD_40P
- added J801: Wurth 8pin Top Contact FPC, Phase2:Wurth_68710814022, symbol Phase2:Wurth_68710814022
- added J901: BL HARD DISABLE, Connector_PinHeader_2.54mm:PinHeader_1x02_P2.54mm_Vertical, symbol Phase2:J901_BL_HARD_DISABLE
- added L201: 2.2uH 8A, Phase2:L_Bourns_SRP1038A_10.0x10.0mm, symbol Phase2:L201_2.2uH_8A
- added L301: 15uH, Inductor_SMD:L_Coilcraft_XAL7070-XXX, symbol Phase2:L301_15uH
- added L501: 10uH, Inductor_SMD:L_Coilcraft_XAL7070-XXX, symbol Phase2:L501_10uH
- added L901: 68uH, Inductor_SMD:L_Vishay_IHLP-6767, symbol Phase2:L901_68uH
- added PWR101: PWR_FLAG, symbol Phase2:PWR101_PWR_FLAG
- added PWR201: PWR_FLAG, symbol Phase2:PWR201_PWR_FLAG
- added PWR301: PWR_FLAG, symbol Phase2:PWR301_PWR_FLAG
- added PWR501: PWR_FLAG, symbol Phase2:PWR501_PWR_FLAG
- added PWR601: PWR_FLAG, symbol Phase2:PWR601_PWR_FLAG
- added Q201, Q202, Q301, Q302, Q303, Q304: CSD19531Q5A, Phase2:Texas_DQJ0008A_VSONP-8, symbol Phase2:CSD19531Q5A
- added Q801: MMBT3904, Package_TO_SOT_SMD:SOT-23, symbol Phase2:Q801_MMBT3904
- added R1001: 100k, Resistor_SMD:R_0603_1608Metric, symbol Phase2:R1001_100k
- added R1002: 100k, Resistor_SMD:R_0603_1608Metric, symbol Phase2:R1002_100k
- added R1003: 100k, Resistor_SMD:R_0603_1608Metric, symbol Phase2:R1003_100k
- added R1004: 100k, Resistor_SMD:R_0603_1608Metric, symbol Phase2:R1004_100k
- added R1005: 47k, Resistor_SMD:R_0603_1608Metric, symbol Phase2:R1005_47k
- added R1006: 10k, Resistor_SMD:R_0603_1608Metric, symbol Phase2:R1006_10k
- added R1007: 2.2k, Resistor_SMD:R_0603_1608Metric, symbol Phase2:R1007_2.2k
- added R201: 1.0R 2W, Resistor_SMD:R_2512_6332Metric, symbol Phase2:R201_1.0R_2W
- added R202: 56.2k 1%, Resistor_SMD:R_0603_1608Metric, symbol Phase2:R202_56.2k_1%
- added R203, R206: 10.0k 1%, Resistor_SMD:R_0603_1608Metric, symbol Phase2:R203_10.0k_1%
- added R204: 100k 1%, Resistor_SMD:R_0603_1608Metric, symbol Phase2:R204_100k_1%
- added R205: 6.49k 1%, Resistor_SMD:R_0603_1608Metric, symbol Phase2:R205_6.49k_1%
- added R301: 20mR 1% 2W, Resistor_SMD:R_2512_6332Metric, symbol Phase2:R301_20mR_1%_2W
- added R302: 100R, Resistor_SMD:R_0402_1005Metric, symbol Phase2:R302_100R
- added R303: 27.4k 1%, Resistor_SMD:R_0603_1608Metric, symbol Phase2:R303_27.4k_1%
- added R304: 93.1k 1%, Resistor_SMD:R_0603_1608Metric, symbol Phase2:R304_93.1k_1%
- added R305: 15.0k 1%, Resistor_SMD:R_0603_1608Metric, symbol Phase2:R305_15.0k_1%
- added R306: 580k 1%, Resistor_SMD:R_0603_1608Metric, symbol Phase2:R306_580k_1%
- added R307: 20.0k 1%, Resistor_SMD:R_0603_1608Metric, symbol Phase2:R307_20.0k_1%
- added R308: 47k, Resistor_SMD:R_0603_1608Metric, symbol Phase2:R308_47k
- added R309: 100R, Resistor_SMD:R_0402_1005Metric, symbol Phase2:R309_100R
- added R501: 100k 0.1%, Resistor_SMD:R_0603_1608Metric, symbol Phase2:R501_100k_0.1%
- added R502: 24.9k 0.1%, Resistor_SMD:R_0603_1608Metric, symbol Phase2:R502_24.9k_0.1%
- added R503: 1.00M 1%, Resistor_SMD:R_0603_1608Metric, symbol Phase2:R503_1.00M_1%
- added R504: 68.1k 1%, Resistor_SMD:R_0603_1608Metric, symbol Phase2:R504_68.1k_1%
- added R505: 549R 1%, Resistor_SMD:R_0603_1608Metric, symbol Phase2:R505_549R_1%
- added R506: 1.05k 1%, Resistor_SMD:R_0603_1608Metric, symbol Phase2:R506_1.05k_1%
- added R507: 100k, Resistor_SMD:R_0603_1608Metric, symbol Phase2:R507_100k
- added R508: 26.7k, Resistor_SMD:R_0603_1608Metric, symbol Phase2:R508_26.7k
- added R509: 47k, Resistor_SMD:R_0603_1608Metric, symbol Phase2:R509_47k
- added R510: 47k, Resistor_SMD:R_0603_1608Metric, symbol Phase2:R510_47k
- added R511: 100k, Resistor_SMD:R_0603_1608Metric, symbol Phase2:R511_100k
- added R512: 100k, Resistor_SMD:R_0603_1608Metric, symbol Phase2:R512_100k
- added R601: 3.3R 2W PULSE, Resistor_SMD:R_2512_6332Metric, symbol Phase2:R601_3.3R_2W_PULSE
- added R602: 1.00M 1%, Resistor_SMD:R_0603_1608Metric, symbol Phase2:R602_1.00M_1%
- added R603: 21.5k 1%, Resistor_SMD:R_0603_1608Metric, symbol Phase2:R603_21.5k_1%
- added R604: 47k, Resistor_SMD:R_0603_1608Metric, symbol Phase2:R604_47k
- added R605: 10k, Resistor_SMD:R_0603_1608Metric, symbol Phase2:R605_10k
- added R606: 47k, Resistor_SMD:R_0603_1608Metric, symbol Phase2:R606_47k
- added R607: 47k, Resistor_SMD:R_0603_1608Metric, symbol Phase2:R607_47k
- added R608: 47k, Resistor_SMD:R_0603_1608Metric, symbol Phase2:R608_47k
- added R609: 47k, Resistor_SMD:R_0603_1608Metric, symbol Phase2:R609_47k
- added R610: 10k, Resistor_SMD:R_0603_1608Metric, symbol Phase2:R610_10k
- added R611: 100k, Resistor_SMD:R_0603_1608Metric, symbol Phase2:R611_100k
- added R701: 0R 0201, Resistor_SMD:R_0201_0603Metric, symbol Phase2:R701_0R_0201
- added R702: 0R 0201, Resistor_SMD:R_0201_0603Metric, symbol Phase2:R702_0R_0201
- added R703: 0R 0201, Resistor_SMD:R_0201_0603Metric, symbol Phase2:R703_0R_0201
- added R704: 0R 0201, Resistor_SMD:R_0201_0603Metric, symbol Phase2:R704_0R_0201
- added R705: 0R 0201, Resistor_SMD:R_0201_0603Metric, symbol Phase2:R705_0R_0201
- added R706: 0R 0201, Resistor_SMD:R_0201_0603Metric, symbol Phase2:R706_0R_0201
- added R801: 100k, Resistor_SMD:R_0603_1608Metric, symbol Phase2:R801_100k
- added R802: 100k, Resistor_SMD:R_0603_1608Metric, symbol Phase2:R802_100k
- added R803: 4.7k, Resistor_SMD:R_0603_1608Metric, symbol Phase2:R803_4.7k
- added R804: 100k, Resistor_SMD:R_0603_1608Metric, symbol Phase2:R804_100k
- added R901: 1.65R 0.1%, Resistor_SMD:R_1206_3216Metric, symbol Phase2:R901_1.65R_0.1%
- added R902: 1.65R 0.1%, Resistor_SMD:R_1206_3216Metric, symbol Phase2:R902_1.65R_0.1%
- added R903: 100R, Resistor_SMD:R_0603_1608Metric, symbol Phase2:R903_100R
- added R904: 83k 1%, Resistor_SMD:R_0603_1608Metric, symbol Phase2:R904_83k_1%
- added R905: 100R, Resistor_SMD:R_0603_1608Metric, symbol Phase2:R905_100R
- added R906: 0R, Resistor_SMD:R_0603_1608Metric, symbol Phase2:R906_0R
- added R907: 1.00M, Resistor_SMD:R_0603_1608Metric, symbol Phase2:R907_1.00M
- added R908: 47k, Resistor_SMD:R_0603_1608Metric, symbol Phase2:R908_47k
- added R909: 100k, Resistor_SMD:R_0603_1608Metric, symbol Phase2:R909_100k
- added R910: 0R LED CURRENT LINK, Resistor_SMD:R_2512_6332Metric, symbol Phase2:R910_0R_LED_CURRENT_LINK
- added TP1001: LCD_PWR_EN, TestPoint:TestPoint_THTPad_D1.0mm_Drill0.5mm, symbol Phase2:TP1001_LCD_PWR_EN
- added TP1002: LCD_RESET_CMD_N, TestPoint:TestPoint_THTPad_D1.0mm_Drill0.5mm, symbol Phase2:TP1002_LCD_RESET_CMD_N
- added TP1003: BL_PWM, TestPoint:TestPoint_THTPad_D1.0mm_Drill0.5mm, symbol Phase2:TP1003_BL_PWM
- added TP1004: CTP_RESET_N_NANO, TestPoint:TestPoint_THTPad_D1.0mm_Drill0.5mm, symbol Phase2:TP1004_CTP_RESET_N_NANO
- added TP1005: CTP_INT_NANO, TestPoint:TestPoint_THTPad_D1.0mm_Drill0.5mm, symbol Phase2:TP1005_CTP_INT_NANO
- added TP1006: GND, TestPoint:TestPoint_THTPad_D1.0mm_Drill0.5mm, symbol Phase2:TP1006_GND
- added TP103: GND, TestPoint:TestPoint_THTPad_D1.0mm_Drill0.5mm, symbol Phase2:TP103_GND
- added TP201: VEH_12V_RAW, TestPoint:TestPoint_THTPad_D1.0mm_Drill0.5mm, symbol Phase2:TP201_VEH_12V_RAW
- added TP202: VEH_PROT, TestPoint:TestPoint_THTPad_D1.0mm_Drill0.5mm, symbol Phase2:TP202_VEH_PROT
- added TP301: SYS_24V, TestPoint:TestPoint_THTPad_D1.0mm_Drill0.5mm, symbol Phase2:TP301_SYS_24V
- added TP302: SYS24_PGOOD, TestPoint:TestPoint_THTPad_D1.0mm_Drill0.5mm, symbol Phase2:TP302_SYS24_PGOOD
- added TP501: SYS_5V_3A, TestPoint:TestPoint_THTPad_D1.0mm_Drill0.5mm, symbol Phase2:TP501_SYS_5V_3A
- added TP502: NANO_5V, TestPoint:TestPoint_THTPad_D1.0mm_Drill0.5mm, symbol Phase2:TP502_NANO_5V
- added TP503: SYS5_PGOOD, TestPoint:TestPoint_THTPad_D1.0mm_Drill0.5mm, symbol Phase2:TP503_SYS5_PGOOD
- added TP504: NANO_EFUSE_FLT, TestPoint:TestPoint_THTPad_D1.0mm_Drill0.5mm, symbol Phase2:TP504_NANO_EFUSE_FLT
- added TP601: VIN_GOOD, TestPoint:TestPoint_THTPad_D1.0mm_Drill0.5mm, symbol Phase2:TP601_VIN_GOOD
- added TP602: SEQ_FLAG1, TestPoint:TestPoint_THTPad_D1.0mm_Drill0.5mm, symbol Phase2:TP602_SEQ_FLAG1
- added TP603: SEQ_FLAG2, TestPoint:TestPoint_THTPad_D1.0mm_Drill0.5mm, symbol Phase2:TP603_SEQ_FLAG2
- added TP604: SEQ_FLAG3, TestPoint:TestPoint_THTPad_D1.0mm_Drill0.5mm, symbol Phase2:TP604_SEQ_FLAG3
- added TP605: LCD_IOVCC, TestPoint:TestPoint_THTPad_D1.0mm_Drill0.5mm, symbol Phase2:TP605_LCD_IOVCC
- added TP606: LCD_VCI, TestPoint:TestPoint_THTPad_D1.0mm_Drill0.5mm, symbol Phase2:TP606_LCD_VCI
- added TP607: LCD_RESET_N, TestPoint:TestPoint_THTPad_D1.0mm_Drill0.5mm, symbol Phase2:TP607_LCD_RESET_N
- added TP801: TOUCH_3V3, TestPoint:TestPoint_THTPad_D1.0mm_Drill0.5mm, symbol Phase2:TP801_TOUCH_3V3
- added TP802: CTP_SCL, TestPoint:TestPoint_THTPad_D1.0mm_Drill0.5mm, symbol Phase2:TP802_CTP_SCL
- added TP803: CTP_SDA, TestPoint:TestPoint_THTPad_D1.0mm_Drill0.5mm, symbol Phase2:TP803_CTP_SDA
- added TP804: CTP_INT, TestPoint:TestPoint_THTPad_D1.0mm_Drill0.5mm, symbol Phase2:TP804_CTP_INT
- added TP805: CTP_RESET_N, TestPoint:TestPoint_THTPad_D1.0mm_Drill0.5mm, symbol Phase2:TP805_CTP_RESET_N
- added TP901: BL_PWM, TestPoint:TestPoint_THTPad_D1.0mm_Drill0.5mm, symbol Phase2:TP901_BL_PWM
- added TP902: BL_DIM, TestPoint:TestPoint_THTPad_D1.0mm_Drill0.5mm, symbol Phase2:TP902_BL_DIM
- added TP903: LED_A, TestPoint:TestPoint_THTPad_D1.0mm_Drill0.5mm, symbol Phase2:TP903_LED_A
- added TP904: LED_K, TestPoint:TestPoint_THTPad_D1.0mm_Drill0.5mm, symbol Phase2:TP904_LED_K
- added TP905: BL_FAULT_N, TestPoint:TestPoint_THTPad_D1.0mm_Drill0.5mm, symbol Phase2:TP905_BL_FAULT_N
- added U201: LM74800QDRRRQ1, Phase2:Texas_DRR0012E_WSON-12_3x3mm_P0.5mm_EP1.3x2.5mm, symbol Phase2:U201_LM74800QDRRRQ1
- added U301: LM5176QPWPRQ1, Phase2:Texas_PWP0028V_TSSOP-28-1EP_4.4x9.7mm_P0.65mm_EP3.4x9.7mm_Mask2.94x5.62mm_ThermalVias, symbol Phase2:U301_LM5176QPWPRQ1
- added U501: LM76003RNPR, Phase2:Texas_RNP0030B_WQFN-30-1EP_4x6mm_P0.5mm_EP1.8x4.5mm_ThermalVias, symbol Phase2:U501_LM76003RNPR
- added U502: TPS259470ARPWR, Phase2:RPW0010A-MFG, symbol Phase2:U502_TPS259470ARPWR
- added U601: TPS3808G01DBVR, Package_TO_SOT_SMD:SOT-23-6, symbol Phase2:U601_TPS3808G01DBVR
- added U602: LM3880MF-1AA/NOPB, Package_TO_SOT_SMD:SOT-23-6, symbol Phase2:U602_LM3880MF-1AA_NOPB
- added U603: TLV75518PDBVR, Package_TO_SOT_SMD:SOT-23-5, symbol Phase2:U603_TLV75518PDBVR
- added U604: TLV75528PDBVR, Package_TO_SOT_SMD:SOT-23-5, symbol Phase2:U604_TLV75528PDBVR
- added U605: TPS22919DCKR, Package_TO_SOT_SMD:SOT-363_SC-70-6, symbol Phase2:U605_TPS22919DCKR
- added U606: SN74LVC1G07DBVR, Package_TO_SOT_SMD:SOT-23-5, symbol Phase2:U606_SN74LVC1G07DBVR
- added U607: SN74LVC1G07DBVR, Package_TO_SOT_SMD:SOT-23-5, symbol Phase2:U607_SN74LVC1G07DBVR
- added U608: SN74LVC1G07DBVR, Package_TO_SOT_SMD:SOT-23-5, symbol Phase2:U608_SN74LVC1G07DBVR
- added U701: TPD6E05U06RVZR, Package_SON:Texas_R-PUSON-N14, symbol Phase2:U701_TPD6E05U06RVZR
- added U801: TLV75533PDBVR, Package_TO_SOT_SMD:SOT-23-5, symbol Phase2:U801_TLV75533PDBVR
- added U802: TMUX1574PWR, Package_SO:TSSOP-16_4.4x5mm_P0.65mm, symbol Phase2:U802_TMUX1574PWR
- added U803: TPD4E05U06DQAR, Package_SON:USON-10_2.5x1.0mm_P0.5mm, symbol Phase2:U803_TPD4E05U06DQAR
- added U901: TPS922053DYYR, Phase2:Texas_DYY0014A_TSOT-23-14, symbol Phase2:U901_TPS922053DYYR
- added U902: SN74LVC1G11DCKR, Package_TO_SOT_SMD:SOT-363_SC-70-6, symbol Phase2:U902_SN74LVC1G11DCKR
Connections:
- new net BL_DIM: J901.2, R909.1, TP902.1 (BL_DIM), U901.6 (EN/PWM)
- new net BL_FAULT_N: J1003.8 (BL_FAULT), R908.1, TP905.1 (BL_FAULT_N), U901.7 (FAULT_N)
- new net BL_GATE_OK: J901.1, U902.4 (Y)
- new net BL_PWM: J1001.7 (GPIO23_BL_PWM), R1003.1, TP1003.1 (BL_PWM), TP901.1 (BL_PWM), U902.1 (A)
- new net BL_SW: D901.2 (A), L901.1, U901.14 (SW)
- new net BOOT1: C307.1, D301.1 (K), U301.26 (BOOT1)
- new net BOOT2: C308.1, D302.1 (K), U301.20 (BOOT2)
- new net BUCK_SHUNT_HI: Q302.1 (S), Q302.2 (S), Q302.3 (S), R301.1, R302.1
- new net BUS_SENSE: C607.1, R602.2, R603.1, U601.5 (SENSE)
- new net COMP_RC: C304.1, R305.2
- new net CTP_INT: J801.6 (INT), R803.1, TP804.1 (CTP_INT), U802.11 (S3A), U803.4 (D2+)
- new net CTP_INT_NANO: J1001.23 (GPIO32_CTP_INT), R1005.1, TP1005.1 (CTP_INT_NANO), U802.9 (D3)
- new net CTP_RESET_N: J801.7 (RST_N), R804.1, TP805.1 (CTP_RESET_N), U802.14 (S4A), U803.5 (D2-)
- new net CTP_RESET_N_NANO: J1001.16 (GPIO22_CTP_RESET), R1004.1, TP1004.1 (CTP_RESET_N_NANO), U802.12 (D4)
- new net CTP_SCL: J801.4 (SCL), TP802.1 (CTP_SCL), U802.2 (S1A), U803.1 (D1+)
- new net CTP_SDA: J801.5 (SDA), TP803.1 (CTP_SDA), U802.5 (S2A), U803.2 (D1-)
- new net DISP_HOLD_5V: C601.1, C603.1, PWR601.1 (PWR_FLAG), R601.2, R604.2, R607.2, R608.2, R609.2, U601.3 (MR_N), U601.6 (VDD), U602.1 (VCC), U603.1 (IN), U604.1 (IN)
- new net DSI_CLK_N_SRC: J701.4 (DSI_CLK_N), R705.1
- new net DSI_CLK_P_SRC: J701.5 (DSI_CLK_P), R706.1
- new net DSI_D0_N_SRC: J701.7 (DSI_D0_N), R701.1
- new net DSI_D0_P_SRC: J701.8 (DSI_D0_P), R702.1
- new net DSI_D1_N_SRC: J701.1 (DSI_D1_N), R703.1
- new net DSI_D1_P_SRC: J701.2 (DSI_D1_P), R704.1
- new net EFUSE_DVDT: C512.1, U502.7 (DVDT)
- new net EFUSE_EN: R511.2, R512.1, U502.1 (EN/UVLO)
- new net EFUSE_ILM: R505.1, R506.1, U502.9 (ILM)
- new net EFUSE_OV: R507.2, R508.1, U502.2 (OVLO)
- new net GND: C201.2, C202.2, C203.2, C204.2, C206.2, C302.2, C303.2, C304.2, C305.2, C306.2, C309.2, C310.2, C311.2, C312.2, C313.2, C502.2, C503.2, C504.2, C505.2, C506.2, C507.2, C508.2, C509.2, C510.2, C511.2, C512.2, C513.2, C514.2, C601.2, C602.2, C603.2, C604.2, C605.2, C606.2, C607.2, C801.2, C802.2, C803.2, C901.2, C902.2, C903.2, C906.2, C907.2, C908.2, D201.2 (A), J1001.14 (GND), J1001.20 (GND), J1001.25 (GND), J1001.6 (GND), J1001.9 (GND), J1002.25 (GND), J1002.26 (GND), J1003.1 (GND), J201.2 (BATT-), J701.13 (GND), J701.3 (GND), J701.6 (GND), J701.9 (GND), J702.10 (GND), J702.13 (GND), J702.16 (GND), J702.17 (GND), J702.18 (GND), J702.19 (GND), J702.20 (GND), J702.21 (GND), J702.22 (GND), J702.25 (GND), J702.30 (GND), J702.4 (GND), J702.7 (GND), J801.1 (GND), J801.8 (GND), PWR101.1 (PWR_FLAG), Q304.1 (S), Q304.2 (S), Q304.3 (S), Q801.2 (E), R1001.2, R1002.2, R1003.2, R1004.2, R1005.2, R1006.2, R1007.2, R203.2, R205.2, R301.2, R303.2, R304.2, R307.2, R309.1, R502.2, R504.2, R505.2, R506.2, R508.2, R512.2, R603.2, R606.2, R611.2, R804.2, R904.2, R907.2, R909.2, TP1006.1 (GND), TP103.1 (GND), U201.7 (GND), U301.10 (AGND), U301.22 (PGND), U301.29 (EP), U301.5 (DITH), U501.13 (AGND), U501.14 (AGND), U501.15 (AGND), U501.17 (SYNC/MODE), U501.19 (NC_GND), U501.23 (NC_GND), U501.24 (PGND), U501.25 (PGND), U501.26 (PGND), U501.27 (NC_GND), U501.28 (NC_GND), U501.29 (NC_GND), U501.30 (NC_GND), U501.31 (EP), U501.7 (NC_GND), U502.8 (GND), U601.2 (GND), U602.2 (GND), U603.2 (GND), U604.2 (GND), U605.2 (GND), U606.3 (GND), U607.3 (GND), U608.3 (GND), U701.10 (GND), U701.5 (GND), U801.2 (GND), U802.1 (SEL), U802.10 (S3B), U802.13 (S4B), U802.3 (S1B), U802.6 (S2B), U802.8 (GND), U803.3 (GND), U803.8 (GND), U901.1 (PGND), U901.2 (AGND), U901.8 (TEMP), U902.3 (GND)
- new net HDRV1: Q301.4 (G), U301.27 (HDRV1)
- new net HDRV2: Q303.4 (G), U301.19 (HDRV2)
- new net HOLD_CHARGE: D601.1 (K), R601.1
- new net LCD_IOVCC: C604.1, J702.3 (IOVCC_1V8), R610.1, TP605.1 (LCD_IOVCC), U603.5 (OUT), U606.5 (VCC), U607.5 (VCC), U608.5 (VCC)
- new net LCD_PWR_EN: J1001.13 (GPIO20_LCD_PWR_EN), R1001.1, R605.1, TP1001.1 (LCD_PWR_EN)
- new net LCD_RESET_CMD_N: J1001.15 (GPIO21_LCD_RESET), R1002.1, TP1002.1 (LCD_RESET_CMD_N), U606.2 (A)
- new net LCD_RESET_N: J1003.7 (LCD_RST), J702.5 (RESET_N), R610.2, R611.1, TP607.1 (LCD_RESET_N), U606.4 (Y_OD), U607.4 (Y_OD), U608.4 (Y_OD)
- new net LCD_VCI: C606.1, J702.2 (VCI_2V8), TP606.1 (LCD_VCI), U605.5 (QOD), U605.6 (VOUT)
- new net LCD_VCI_RAW: C605.1, U604.5 (OUT), U605.1 (VIN)
- new net LDRV1: Q302.4 (G), U301.25 (LDRV1)
- new net LDRV2: Q304.4 (G), U301.21 (LDRV2)
- new net LED24_R: D1001.1 (K), R1006.1
- new net LED5_R: D1002.1 (K), R1007.1
- new net LED_A: C905.1, C908.1, FB901.2, J702.39 (LED+), J702.40 (LED+), TP903.1 (LED_A)
- new net LED_K: C905.2, J702.31 (LED-), J702.32 (LED-), R906.1, R910.1, TP904.1 (LED_K)
- new net LED_K_RAW: R901.1, R902.1, R903.1, R910.2
- new net LED_SENSE_N: C904.2, L901.2, R901.2, R902.2, U901.13 (CSN)
- new net LM5176_COMP: C305.1, R305.1, U301.9 (COMP)
- new net LM5176_CS: C301.1, R302.2, U301.16 (CS)
- new net LM5176_CSG: C301.2, R309.2, U301.15 (CSG)
- new net LM5176_MODE: R304.1, U301.4 (MODE)
- new net LM5176_RT: R303.1, U301.6 (RT/SYNC)
- new net LM5176_SLOPE: C302.1, U301.7 (SLOPE)
- new net LM5176_SS: C303.1, U301.8 (SS)
- new net LM5176_VCC: C306.1, D301.2 (A), D302.2 (A), U301.23 (VCC)
- new net LM760_BOOT: C501.1, U501.6 (BOOT)
- new net LM760_EN: R503.2, R504.1, U501.18 (EN)
- new net LM760_FB: R501.2, R502.1, U501.12 (FB)
- new net LM760_SS: C504.1, U501.11 (SS/TRK)
- new net LM760_SW: C501.2, L501.1, U501.1 (SW), U501.2 (SW), U501.3 (SW), U501.4 (SW), U501.5 (SW)
- new net LM760_VCC: C502.1, U501.8 (VCC)
- new net MIPI_0N: J702.8 (MIPI_0N), R701.2, U701.14 (D1+)
- new net MIPI_0P: J702.9 (MIPI_0P), R702.2, U701.13 (D1-)
- new net MIPI_1N: J702.11 (MIPI_1N), R703.2, U701.12 (D2+)
- new net MIPI_1P: J702.12 (MIPI_1P), R704.2, U701.11 (D2-)
- new net MIPI_CLKN: J702.14 (MIPI_CLKN), R705.2, U701.9 (D3+)
- new net MIPI_CLKP: J702.15 (MIPI_CLKP), R706.2, U701.8 (D3-)
- new net NANO_3V3_DETECT: Q801.1 (B), R801.2
- new net NANO_3V3_REF: J701.14 (ESP_3V3_REF), J701.15 (ESP_3V3_REF), R801.1
- new net NANO_5V: J1001.2 (5V), J1001.4 (5V), J501.2, TP502.1 (NANO_5V)
- new net NANO_5V_EFUSED: C514.1, J501.1, U502.6 (OUT)
- new net NANO_EFUSE_FLT: J1003.9 (5V_FAULT), R509.1, TP504.1 (NANO_EFUSE_FLT), U502.4 (FLT)
- new net NANO_I2C_SCL: J701.11 (GPIO8_I2C_SCL), U802.4 (D1)
- new net NANO_I2C_SDA: J701.12 (GPIO7_I2C_SDA), U802.7 (D2)
- new net SEQ_ENABLE: D602.2 (A), R605.2, R606.1, U602.3 (EN)
- new net SEQ_FLAG1: J1003.4 (SEQ1), R607.1, TP602.1 (SEQ_FLAG1), U602.6 (FLAG1), U603.3 (EN), U604.3 (EN)
- new net SEQ_FLAG2: J1003.5 (SEQ2), R608.1, TP603.1 (SEQ_FLAG2), U602.5 (FLAG2), U605.3 (ON)
- new net SEQ_FLAG3: J1003.6 (SEQ3), R609.1, TP604.1 (SEQ_FLAG3), U602.4 (FLAG3), U607.2 (A), U902.2 (B)
- new net SW1: C307.2, L301.1, Q301.1 (S), Q301.2 (S), Q301.3 (S), Q302.5 (D), Q302.6 (D), Q302.7 (D), Q302.8 (D), U301.28 (SW1)
- new net SW2: C308.2, L301.2, Q303.1 (S), Q303.2 (S), Q303.3 (S), Q304.5 (D), Q304.6 (D), Q304.7 (D), Q304.8 (D), U301.18 (SW2)
- new net SYS24_PGOOD: J1003.10 (SYS24_PGOOD), R308.1, TP302.1 (SYS24_PGOOD), U301.17 (PGOOD)
- new net SYS5_PGOOD: R510.1, TP503.1 (SYS5_PGOOD), U501.16 (PGOOD)
- new net SYS_24V: C311.1, C312.1, C313.1, C505.1, C506.1, C507.1, C901.1, C902.1, D1001.2 (A), D901.1 (K), FB901.1, PWR301.1 (PWR_FLAG), Q303.5 (D), Q303.6 (D), Q303.7 (D), Q303.8 (D), R306.1, R503.1, R602.1, TP301.1 (SYS_24V), U301.12 (VOSNS), U301.13 (ISNS-), U301.14 (ISNS+), U301.24 (BIAS), U501.20 (PVIN), U501.21 (PVIN), U501.22 (PVIN), U901.3 (VIN)
- new net SYS_5V_3A: C503.1, C508.1, C509.1, C510.1, C511.1, C513.1, C801.1, D1002.2 (A), D601.2 (A), J1003.2 (5V), L501.2, PWR501.1 (PWR_FLAG), R308.2, R501.1, R507.1, R509.2, R510.2, R511.1, TP501.1 (SYS_5V_3A), U501.9 (BIAS), U502.5 (IN), U801.1 (IN)
- new net TMUX_EN_N: Q801.3 (C), R802.1, U802.15 (EN_N)
- new net TOUCH_3V3: C802.1, C803.1, J801.3 (VDD_3V3), R802.2, R803.2, TP801.1 (TOUCH_3V3), U801.5 (OUT), U802.16 (VDD), U902.6 (VCC)
- new net TPS3808_CT: C602.1, U601.4 (CT)
- new net TPS922_COMP: C906.1, R905.1, U901.10 (COMP)
- new net TPS922_COMP_C: C907.1, R905.2
- new net TPS922_CSP: C904.1, R903.2, U901.12 (CSP)
- new net TPS922_FSET: R904.1, U901.9 (FSET)
- new net TPS922_UVP: R906.2, R907.1, U901.11 (UVP)
- new net TPS922_VCC: C903.1, R908.2, U901.4 (VCC), U901.5 (ADIM/HD)
- new net VEH_12V_RAW: F201.1, J201.1 (BATT+), TP201.1 (VEH_12V_RAW)
- new net VEH_CAP: C205.1, U201.11 (CAP)
- new net VEH_DAMP: C204.1, R201.2
- new net VEH_DGATE: Q201.4 (G), U201.1 (DGATE)
- new net VEH_FB: R306.2, R307.1, U301.11 (FB)
- new net VEH_FET_MID: C205.2, C206.1, Q201.5 (D), Q201.6 (D), Q201.7 (D), Q201.8 (D), Q202.5 (D), Q202.6 (D), Q202.7 (D), Q202.8 (D), U201.10 (VS), U201.12 (C)
- new net VEH_FILTER: C201.1, C202.1, D201.1 (K), L201.2, Q201.1 (S), Q201.2 (S), Q201.3 (S), R201.1, R202.1, U201.2 (A), U201.3 (VSNS)
- new net VEH_FUSED: F201.2, L201.1
- new net VEH_HGATE: Q202.4 (G), R206.1, U201.8 (HGATE)
- new net VEH_HGATE_DVDT: C207.1, R206.2
- new net VEH_OV: R204.2, R205.1, U201.5 (OV)
- new net VEH_OV_TOP: R204.1, U201.4 (SW)
- new net VEH_PROT: C203.1, C207.2, C309.1, C310.1, PWR201.1 (PWR_FLAG), Q202.1 (S), Q202.2 (S), Q202.3 (S), Q301.5 (D), Q301.6 (D), Q301.7 (D), Q301.8 (D), TP202.1 (VEH_PROT), U201.9 (OUT), U301.1 (EN/UVLO), U301.2 (VIN), U301.3 (VISNS)
- new net VEH_UVLO: R202.2, R203.1, U201.6 (EN/UVLO)
- new net VIN_GOOD: D602.1 (K), J1003.3 (VIN_GOOD), R604.1, TP601.1 (VIN_GOOD), U601.1 (RESET_N), U608.2 (A), U801.3 (EN), U902.5 (C)
- no-connect marks 0 -> 55
Other:
- removed sheet Display Power & Backlight
- removed sheet Interfaces & Nano
- removed sheet Power
- note added: "01: SINGLE 12 V INPUT"
- note added: "02: VEHICLE INPUT PROTECTION"
- note added: "03: LM5176 SINGLE-SOURCE BUCK-BOOST"
- note added: "05: SYSTEM 5 V AND NANO FEED"
- note added: "06: DISPLAY RAILS AND SEQUENCING"
- note added: "07: MIPI DSI AND LCD CONNECTOR"
- note added: "08: GT9271 TOUCH INTERFACE"
- note added: "09: 240 MA BACKLIGHT"
- note added: "100k/24.9k feedback gives 5.016 V nominal. 22 nF SS gives approximately 11 ms ramp."
- note added: "10: NANO HEADERS AND DEBUG"
- note added: "6800 uF is isolated from Nano/backlight. At 0.20 A for 30 ms, droop is 0.88 V; sequencing remains above LDO dropout."
- note added: "83k FSET selects 300 kHz. 68 uH is validated over the regulated SYS_24V range; see calculations."
- note added: "At 8 V/30 W/85%, Iavg=4.41 A. With 15 uH, ripple is about 1.19 App and peak about 5.00 A."
- note added: "Bench development uses a regulated/current-limited nominal 12 V supply at J201."
- note added: "Corrected P1 controls: pin 7 GPIO23 BL PWM; 13 GPIO20 LCD power; 15 GPIO21 LCD reset; 16 GPIO22 touch reset; 23 GPIO32 touch INT."
- note added: "F101/TVS coordination and adapter inrush are prototype verification items; no automotive qualification claim."
- note added: "LM5176 output directly supplies SYS_24V; no high-voltage source ORing is present."
- note added: "LM76003: 500 kHz, 10 uH; checked over the regulated SYS_24V range. 4x22 uF output bank."
- note added: "Nano I2C already has 2.2k pull-ups; no additional Nano-side pull-ups. Touch INT has the vendor-required 4.7k pull-up."
- note added: "OV divider 100k/6.49k: 20.18 V nominal cutoff; rejects accidental 24 V vehicle-port connection."
- note added: "P1 pins 2/4 are Nano 5 V. GPIO21/P1-13 is an unconnected documented alternate. GPIO24 remains untouched for USB Serial/JTAG."
- note added: "R701–R706 are inline zero-ohm 0201 tuning locations; layout them as minimal-discontinuity pass-through pads."
- note added: "SYSTEM 24 V DISTRIBUTION (DEPRECATED)"
- note added: "SYS_24V has 264 uF converter output capacitance plus 19.547 uF distributed local bypass."
- note added: "Straight-through lane identity and polarity. No AC coupling, common-mode choke, probe pad, or branch."
- note added: "TMUX1574 SEL=0 uses the A paths; all B paths are grounded per datasheet. EN_N is pulled high when Nano 3.3 V is absent."
- note added: "TPS3808 threshold: 0.405*(1M+21.5k)/21.5k = 19.23 V nominal. Its reset directly clamps sequence/reset/backlight validity."
- note added: "Target: 24.0 V, 30 W continuous, 300 kHz. RFB 580k/20k gives 24.0 V nominal."
- note added: "Two 1.65 ohm/0.1% resistors in parallel give 0.825 ohm: 242.4 mA nominal; +3% threshold gives 249.9 mA."
- note added: "UVLO divider 56.2k/10.0k: 8.15 V rising, about 7.49 V falling using LM7480 thresholds."
- note removed: "PHASE 2 SCHEMATIC — PCB layout not started. Native KiCad files are authoritative."

Commit message: design update
Parts:
- removed J1003: DEBUG HEADER, Connector_PinHeader_2.54mm:PinHeader_2x05_P2.54mm_Vertical, symbol Phase2:J1003_DEBUG_HEADER
- removed TP1001: LCD_PWR_EN, TestPoint:TestPoint_THTPad_D1.0mm_Drill0.5mm, symbol Phase2:TP1001_LCD_PWR_EN
- removed TP1002: LCD_RESET_CMD_N, TestPoint:TestPoint_THTPad_D1.0mm_Drill0.5mm, symbol Phase2:TP1002_LCD_RESET_CMD_N
- removed TP1003: BL_PWM, TestPoint:TestPoint_THTPad_D1.0mm_Drill0.5mm, symbol Phase2:TP1003_BL_PWM
- removed TP1004: CTP_RESET_N_NANO, TestPoint:TestPoint_THTPad_D1.0mm_Drill0.5mm, symbol Phase2:TP1004_CTP_RESET_N_NANO
- removed TP1005: CTP_INT_NANO, TestPoint:TestPoint_THTPad_D1.0mm_Drill0.5mm, symbol Phase2:TP1005_CTP_INT_NANO
- removed TP1006: GND, TestPoint:TestPoint_THTPad_D1.0mm_Drill0.5mm, symbol Phase2:TP1006_GND
- removed TP103: GND, TestPoint:TestPoint_THTPad_D1.0mm_Drill0.5mm, symbol Phase2:TP103_GND
- removed TP201: VEH_12V_RAW, TestPoint:TestPoint_THTPad_D1.0mm_Drill0.5mm, symbol Phase2:TP201_VEH_12V_RAW
- removed TP202: VEH_PROT, TestPoint:TestPoint_THTPad_D1.0mm_Drill0.5mm, symbol Phase2:TP202_VEH_PROT
- removed TP301: SYS_24V, TestPoint:TestPoint_THTPad_D1.0mm_Drill0.5mm, symbol Phase2:TP301_SYS_24V
- removed TP302: SYS24_PGOOD, TestPoint:TestPoint_THTPad_D1.0mm_Drill0.5mm, symbol Phase2:TP302_SYS24_PGOOD
- removed TP501: SYS_5V_3A, TestPoint:TestPoint_THTPad_D1.0mm_Drill0.5mm, symbol Phase2:TP501_SYS_5V_3A
- removed TP502: NANO_5V, TestPoint:TestPoint_THTPad_D1.0mm_Drill0.5mm, symbol Phase2:TP502_NANO_5V
- removed TP503: SYS5_PGOOD, TestPoint:TestPoint_THTPad_D1.0mm_Drill0.5mm, symbol Phase2:TP503_SYS5_PGOOD
- removed TP504: NANO_EFUSE_FLT, TestPoint:TestPoint_THTPad_D1.0mm_Drill0.5mm, symbol Phase2:TP504_NANO_EFUSE_FLT
- removed TP601: VIN_GOOD, TestPoint:TestPoint_THTPad_D1.0mm_Drill0.5mm, symbol Phase2:TP601_VIN_GOOD
- removed TP602: SEQ_FLAG1, TestPoint:TestPoint_THTPad_D1.0mm_Drill0.5mm, symbol Phase2:TP602_SEQ_FLAG1
- removed TP603: SEQ_FLAG2, TestPoint:TestPoint_THTPad_D1.0mm_Drill0.5mm, symbol Phase2:TP603_SEQ_FLAG2
- removed TP604: SEQ_FLAG3, TestPoint:TestPoint_THTPad_D1.0mm_Drill0.5mm, symbol Phase2:TP604_SEQ_FLAG3
- removed TP605: LCD_IOVCC, TestPoint:TestPoint_THTPad_D1.0mm_Drill0.5mm, symbol Phase2:TP605_LCD_IOVCC
- removed TP606: LCD_VCI, TestPoint:TestPoint_THTPad_D1.0mm_Drill0.5mm, symbol Phase2:TP606_LCD_VCI
- removed TP607: LCD_RESET_N, TestPoint:TestPoint_THTPad_D1.0mm_Drill0.5mm, symbol Phase2:TP607_LCD_RESET_N
- removed TP801: TOUCH_3V3, TestPoint:TestPoint_THTPad_D1.0mm_Drill0.5mm, symbol Phase2:TP801_TOUCH_3V3
- removed TP802: CTP_SCL, TestPoint:TestPoint_THTPad_D1.0mm_Drill0.5mm, symbol Phase2:TP802_CTP_SCL
- removed TP803: CTP_SDA, TestPoint:TestPoint_THTPad_D1.0mm_Drill0.5mm, symbol Phase2:TP803_CTP_SDA
- removed TP804: CTP_INT, TestPoint:TestPoint_THTPad_D1.0mm_Drill0.5mm, symbol Phase2:TP804_CTP_INT
- removed TP805: CTP_RESET_N, TestPoint:TestPoint_THTPad_D1.0mm_Drill0.5mm, symbol Phase2:TP805_CTP_RESET_N
- removed TP901: BL_PWM, TestPoint:TestPoint_THTPad_D1.0mm_Drill0.5mm, symbol Phase2:TP901_BL_PWM
- removed TP902: BL_DIM, TestPoint:TestPoint_THTPad_D1.0mm_Drill0.5mm, symbol Phase2:TP902_BL_DIM
- removed TP903: LED_A, TestPoint:TestPoint_THTPad_D1.0mm_Drill0.5mm, symbol Phase2:TP903_LED_A
- removed TP904: LED_K, TestPoint:TestPoint_THTPad_D1.0mm_Drill0.5mm, symbol Phase2:TP904_LED_K
- removed TP905: BL_FAULT_N, TestPoint:TestPoint_THTPad_D1.0mm_Drill0.5mm, symbol Phase2:TP905_BL_FAULT_N
- C207: value 82nF 25V X7R -> 82nF 100V X7R; MPN C0603C823K3RACTU -> C0603C823K1RACAUTO
- R206: value 10.0k 1% -> 100R 1%; MPN ERJ-3EKF1002V -> ERJ-3EKF1000V
Connections:
- net GND: now also C207.2
- net SYS_24V: no longer U301.13 (ISNS-), U301.14 (ISNS+)
- net VEH_PROT: no longer C207.2
- new net: U301.13 (ISNS-), U301.14 (ISNS+)
Other:
- moved on the sheet: D1001, D1002, J1001, J1002, R1001, R1002, R1003, R1004, R1005, R1006, R1007

Commit message: create new firmware for waveshare 8.8" display with touch
Parts:
- removed J1001: SSQ-113-01-G-D, Phase2:Samtec_SSQ-113-01-G-D_BottomMount, symbol Phase2:J1001_NANO_P1_2x13
- removed J1002: SSQ-113-01-G-D, Phase2:Samtec_SSQ-113-01-G-D_BottomMount, symbol Phase2:J1002_NANO_P2_2x13
- removed J701: NANO DSI 15P, Phase2:Amphenol_CON15_1X15_DRB_SFW_FCI, symbol Phase2:J701_NANO_DSI_15P
- added J1: 5034802200, Phase2:CON_5034802200_MOL, symbol Phase2:5034802200
- added J101: ESP32-P4-WIFI6-DB-P1, PCM_SF-Connector:1x20, symbol Phase2:J101_HOST_P1_1X20
- added J102: ESP32-P4-WIFI6-DB-P2, PCM_SF-Connector:1x20, symbol Phase2:J102_HOST_P2_1X20
- added J2: 525592253, Phase2:CON_525592253_MOL, symbol Phase2:525592253
Connections:
- net BL_PWM: now also J101.10 (GPIO23)
- net DSI_CLK_N_SRC: now also J1.15
- net DSI_CLK_P_SRC: now also J1.14
- net DSI_D0_N_SRC: now also J1.21
- net DSI_D0_P_SRC: now also J1.20
- net DSI_D1_N_SRC: now also J1.18
- net DSI_D1_P_SRC: now also J1.17
- net GND: now also J1.10, J1.13, J1.16, J1.19, J1.22, J1.4, J1.7, J101.13 (GND), J101.18 (GND), J101.3 (GND), J101.8 (GND), J102.13 (GND), J102.16 (SCL/GPIO8), J102.18 (GND), J102.3 (GND), J102.8 (GND)
- net LCD_PWR_EN: now also J101.6 (GPIO20)
- net LCD_RESET_CMD_N: now also J101.7 (GPIO21)
- net CTP_INT_NANO renamed CTP_INT_HOST
- net CTP_INT_HOST: now also J101.15 (GPIO32)
- net CTP_RESET_N_NANO renamed CTP_RESET_N_HOST
- net CTP_RESET_N_HOST: now also J101.9 (GPIO22)
- net NANO_3V3_DETECT renamed HOST_3V3_DETECT
- net NANO_3V3_REF renamed HOST_3V3_REF
- net HOST_3V3_REF: now also J1.1
- net NANO_5V renamed HOST_5V
- net HOST_5V: now also J101.2 (VSYS)
- net NANO_5V_EFUSED renamed HOST_5V_EFUSED
- net NANO_EFUSE_FLT renamed HOST_EFUSE_FLT
- net NANO_I2C_SCL renamed HOST_I2C_SCL
- net HOST_I2C_SCL: now also J1.3
- net NANO_I2C_SDA renamed HOST_I2C_SDA
- net HOST_I2C_SDA: now also J1.2
- no-connect marks 55 -> 46
Other:
- note added: "05: SYSTEM 5 V AND HOST FEED"
- note added: "10: HOST HEADERS AND DEBUG"
- note added: "6800 uF is isolated from Host/backlight. At 0.20 A for 30 ms, droop is 0.88 V; sequencing remains above LDO dropout."
- note added: "Host I2C already has 2.2k pull-ups; no additional Host-side pull-ups. Touch INT has the vendor-required 4.7k pull-up."
- note added: "P1 pins 2/4 are Host 5 V. GPIO21/P1-13 is an unconnected documented alternate. GPIO24 remains untouched for USB Serial/JTAG."
- note added: "TMUX1574 SEL=0 uses the A paths; all B paths are grounded per datasheet. EN_N is pulled high when Host 3.3 V is absent."
- note removed: "05: SYSTEM 5 V AND NANO FEED"
- note removed: "10: NANO HEADERS AND DEBUG"
- note removed: "6800 uF is isolated from Nano/backlight. At 0.20 A for 30 ms, droop is 0.88 V; sequencing remains above LDO dropout."
- note removed: "Nano I2C already has 2.2k pull-ups; no additional Nano-side pull-ups. Touch INT has the vendor-required 4.7k pull-up."
- note removed: "P1 pins 2/4 are Nano 5 V. GPIO21/P1-13 is an unconnected documented alternate. GPIO24 remains untouched for USB Serial/JTAG."
- note removed: "TMUX1574 SEL=0 uses the A paths; all B paths are grounded per datasheet. EN_N is pulled high when Nano 3.3 V is absent."
- moved on the sheet: C301, C302, C303, C304, C305, C306, C307, C308, C309, C310, C311, C312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
