File: hardware/kicad/01_power.kicad_sch (KiCad schematic)
At the start: 117 parts, among them J101 RAPC722X 24V BENCH, J201 VEHICLE 12V, J501 SERVICE LINK 5V, Q201 CSD19531Q5A, Q202 CSD19531Q5A, Q301 CSD19531Q5A, Q302 CSD19531Q5A, Q303 CSD19531Q5A, Q304 CSD19531Q5A, Q401 CSD19531Q5A, Q402 CSD19531Q5A, U201 LM74800QDRRRQ1, U301 LM5176QPWPRQ1, U401 LM74700QDBVRQ1, U402 LM74700QDBVRQ1, U501 LM76003RNPR, U502 TPS259470ARPWR

Commit message: hardware: correct audited power startup and schematic geometry
Parts:
- added C207: 82nF 25V X7R, Capacitor_SMD:C_0603_1608Metric, symbol Phase2:C304_82nF_X7R
- added R206: 10.0k 1%, Resistor_SMD:R_0603_1608Metric, symbol Phase2:R203_10.0k_1%
Connections:
- net VEH_FILTER: no longer C203.1
- net VEH_HGATE: now also R206.1
- net VEH_PROT: now also C203.1, C207.2
- new net VEH_HGATE_DVDT: C207.1, R206.2

Commit message: Simplify power architecture to single 12V input
Parts:
- removed C101: 100nF 100V X7R, Capacitor_SMD:C_0603_1608Metric, symbol Phase2:C101_100nF_100V_X7R
- removed C102: 10uF 50V, Capacitor_SMD:C_1210_3225Metric, symbol Phase2:C102_10uF_50V
- removed C103: 47uF 50V, Capacitor_SMD:CP_Elec_8x10, symbol Phase2:C103_47uF_50V
- removed C401: 100nF 25V, Capacitor_SMD:C_0603_1608Metric, symbol Phase2:C401_100nF_25V
- removed C402: 100nF 25V, Capacitor_SMD:C_0603_1608Metric, symbol Phase2:C402_100nF_25V
- removed C403: 220uF 50V, Capacitor_SMD:CP_Elec_10x12.5, symbol Phase2:C403_220uF_50V
- removed C404: 10uF 50V, Capacitor_SMD:C_1210_3225Metric, symbol Phase2:C404_10uF_50V
- removed C405: 22nF 100V, Capacitor_SMD:C_0603_1608Metric, symbol Phase2:C405_22nF_100V
- removed C406: 22nF 100V, Capacitor_SMD:C_0603_1608Metric, symbol Phase2:C406_22nF_100V
- removed C407: 100nF 50V, Capacitor_SMD:C_0603_1608Metric, symbol Phase2:C407_100nF_50V
- removed C408: 100nF 50V, Capacitor_SMD:C_0603_1608Metric, symbol Phase2:C408_100nF_50V
- removed D101: SMBJ30A, Diode_SMD:D_SMB, symbol Phase2:D101_SMBJ30A
- removed F101: 2A FAST, Fuse:Fuse_1206_3216Metric, symbol Phase2:F101_2A_FAST
- removed J101: RAPC722X 24V BENCH, Phase2:Switchcraft_RAPC722X_RightAngle, symbol Phase2:J101_RAPC722X_24V_BENCH
- removed PWR401: PWR_FLAG, symbol Phase2:PWR401_PWR_FLAG
- removed Q401: CSD19531Q5A, Package_SON:Texas_DQK, symbol Phase2:Q401_CSD19531Q5A
- removed Q402: CSD19531Q5A, Package_SON:Texas_DQK, symbol Phase2:Q402_CSD19531Q5A
- removed R401: 0R, Resistor_SMD:R_2512_6332Metric, symbol Phase2:R401_0R
- removed R402: 0R, Resistor_SMD:R_2512_6332Metric, symbol Phase2:R402_0R
- removed TP101: BENCH_24V_RAW, TestPoint:TestPoint_THTPad_D1.0mm_Drill0.5mm, symbol Phase2:TP101_BENCH_24V_RAW
- removed TP102: BENCH_FUSED_24V, TestPoint:TestPoint_THTPad_D1.0mm_Drill0.5mm, symbol Phase2:TP102_BENCH_FUSED_24V
- removed TP401: VIN_PROT_24V, TestPoint:TestPoint_THTPad_D1.0mm_Drill0.5mm, symbol Phase2:TP401_VIN_PROT_24V
- removed TP402: BENCH_OR_24V, TestPoint:TestPoint_THTPad_D1.0mm_Drill0.5mm, symbol Phase2:TP402_BENCH_OR_24V
- removed TP403: VEH_OR_24V, TestPoint:TestPoint_THTPad_D1.0mm_Drill0.5mm, symbol Phase2:TP403_VEH_OR_24V
- removed U401: LM74700QDBVRQ1, Package_TO_SOT_SMD:SOT-23-6, symbol Phase2:U401_LM74700QDBVRQ1
- removed U402: LM74700QDBVRQ1, Package_TO_SOT_SMD:SOT-23-6, symbol Phase2:U402_LM74700QDBVRQ1
- TP301: value VEH_24V -> SYS_24V; symbol Phase2:TP301_VEH_24V -> Phase2:TP301_SYS_24V
- TP302: value VEH_PGOOD -> SYS24_PGOOD; symbol Phase2:TP302_VEH_PGOOD -> Phase2:TP302_SYS24_PGOOD
Connections:
- net VIN_PROT_24V is gone; now on net SYS_24V: C505.1, C506.1, C507.1, R503.1, U501.20 (PVIN), U501.21 (PVIN), U501.22 (PVIN)
- net VEH_24V renamed SYS_24V
- net VEH_PGOOD renamed SYS24_PGOOD
- no-connect marks 2 -> 1
Other:
- note added: "Bench development uses a regulated/current-limited nominal 12 V supply at J201."
- note added: "LM5176 SINGLE-SOURCE BUCK-BOOST"
- note added: "LM5176 output directly supplies SYS_24V; no high-voltage source ORing is present."
- note added: "LM76003: 500 kHz, 10 uH; checked over the regulated SYS_24V range. 4x22 uF output bank."
- note added: "SINGLE 12 V INPUT"
- note added: "SYSTEM 24 V DISTRIBUTION"
- note added: "SYS_24V has 264 uF converter output capacitance plus 19.547 uF distributed local bypass."
- note removed: "BENCH 24 V INPUT"
- note removed: "Each branch has independent LM74700 reverse-current blocking; simultaneous sources are legal."
- note removed: "LM5176 VEHICLE BUCK-BOOST"
- note removed: "LM76003: 500 kHz, 10 uH; ripple about 0.81 App at 26.4 V/3 A. 4x22 uF output bank."
- note removed: "No active current sharing is claimed. The source with the higher delivered voltage supplies the common bus."
- note removed: "Regulated 24 V bench input: 21.6–26.4 V. Center positive."
- note removed: "SOURCE ORING"
- moved on the sheet: TP302
