File: hardware/kicad/02_display_power_backlight.kicad_sch (KiCad schematic)
At the start: 64 parts, among them J901 BL HARD DISABLE, U601 TPS3808G01DBVR, U602 LM3880MF-1AA/NOPB, U603 TLV75518PDBVR, U604 TLV75528PDBVR, U605 TPS22919DCKR, U606 SN74LVC1G07DBVR, U607 SN74LVC1G07DBVR, U608 SN74LVC1G07DBVR, U901 TPS922053DYYR, U902 SN74LVC1G11DCKR

Commit message: hardware: correct audited power startup and schematic geometry
Parts:
- added C607: 1nF 50V C0G, Capacitor_SMD:C_0603_1608Metric, symbol Phase2:C602_100pF_C0G
Connections:
- net BUS_SENSE: now also C607.1
- net GND: now also C607.2

Commit message: Simplify power architecture to single 12V input
Connections:
- net VIN_PROT_24V renamed SYS_24V
Other:
- note added: "83k FSET selects 300 kHz. 68 uH is validated over the regulated SYS_24V range; see calculations."
- note removed: "83k FSET selects 300 kHz. 68 uH gives about 243 mApp ripple at 26.4 V; worst-normal peak about 371 mA."
Changed lines of the file:
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@@
 	(title_block
 		(title "Display Power & Backlight")
-		(date "2026-09-18")
-		(rev "Phase 2 / audit correction v0.3")
+		(date "2026-09-19")
+		(rev "Phase 2 / single-source v0.4")
 		(company "ESP32-P4 Displayman Development Daughterboard")
 		(comment 1 "© 2026 Sy Aryeh")
@@
 		(comment 3 "REV1 development hardware")
 	)
-	(text "83k FSET selects 300 kHz. 68 uH gives about 243 mApp ripple at 26.4 V; worst-normal peak about 371 mA."
+	(text "83k FSET selects 300 kHz. 68 uH is validated over the regulated SYS_24V range; see calculations."
 		(exclude_from_sim no)
 		(at 17.54 305.16 0)
@@
 		)
 	)
-	(global_label "VIN_PROT_24V"
+	(global_label "SYS_24V"
 		(shape bidirectional)
 		(at 789.94 374.65 180)
@@
 		)
 	)
-	(global_label "VIN_PROT_24V"
+	(global_label "SYS_24V"
 		(shape bidirectional)
 		(at 20.32 430.53 180)
@@
 		)
 	)
-	(global_label "VIN_PROT_24V"
+	(global_label "SYS_24V"
 		(shape bidirectional)
 		(at 144.78 374.65 180)
@@
 		)
 	)
-	(global_label "VIN_PROT_24V"
+	(global_label "SYS_24V"
 		(shape bidirectional)
 		(at 144.78 490.22 180)
@@
 		)
 	)
-	(global_label "VIN_PROT_24V"
+	(global_label "SYS_24V"
 		(shape bidirectional)
 		(at 189.23 48.26 180)
@@
 		)
 	)
-	(global_label "VIN_PROT_24V"
+	(global_label "SYS_24V"
 		(shape bidirectional)
 		(at 144.78 317.5 180)
