File: hardware/kicad/ESP32-P4 Display Development Daughterboard.kicad_pcb (KiCad board)
At the start: 2 copper layers, 0 parts

Commit message: updated the background tech drawings and added annotations
Other:
- board text added: "Technical drawings derived from Waveshare ESP32-P4-NANO manufacturer DXF; edited/rescaled for KiCad import. Verify against original vendor PDF/DXF/STEP before mechanical freeze."

Commit message: added board outline with cutouts for ethernet usb and DSI passthrough
Inserted positioned and locked into the Edge Cuts layer approximately matching the Nano drawing on the User 1 layer.
Other:
- board outline added: 85 x 80 mm
