File: hardware/kicad_flux_branch/ESP32-P4 Display FLUX.kicad_sch (KiCad schematic)
At the start: 93 parts, among them J201 VEHICLE 12V, J501 SERVICE LINK 5V, Q201 CSD19531Q5A, Q202 CSD19531Q5A, Q301 CSD19531Q5A, Q302 CSD19531Q5A, Q303 CSD19531Q5A, Q304 CSD19531Q5A, U201 LM74800QDRRRQ1, U301 LM5176QPWPRQ1, U501 LM76003RNPR, U502 TPS259470ARPWR

Commit message: Major fixes. Needs simplification, component organization and routing
Parts:
- removed Q201: CSD19531Q5A, Package_SON:Texas_DQK, symbol Phase2:Q201_CSD19531Q5A
- removed Q202: CSD19531Q5A, Package_SON:Texas_DQK, symbol Phase2:Q202_CSD19531Q5A
- removed Q301: CSD19531Q5A, Package_SON:Texas_DQK, symbol Phase2:Q301_CSD19531Q5A
- removed Q302: CSD19531Q5A, Package_SON:Texas_DQK, symbol Phase2:Q302_CSD19531Q5A
- removed Q303: CSD19531Q5A, Package_SON:Texas_DQK, symbol Phase2:Q303_CSD19531Q5A
- removed Q304: CSD19531Q5A, Package_SON:Texas_DQK, symbol Phase2:Q304_CSD19531Q5A
- added Q201, Q202, Q301, Q302, Q303, Q304: CSD19531Q5A, Phase2:Texas_DQJ0008A_VSONP-8, symbol Phase2:CSD19531Q5A
- J201: footprint Phase2:Molex_Micro-Fit_3.0_43045-0218_2x01-1MP_P3.00mm_Vertical -> Phase2:CONN_SD-43045-007_02_MOL
- U502: footprint Phase2:Texas_RPW0010A_VQFN-HR-10_2x2mm -> Phase2:RPW0010A-MFG
Connections:
- net BUCK_SHUNT_HI: now also Q302.1 (S), Q302.2 (S), Q302.3 (S)
- net GND: now also Q304.1 (S), Q304.2 (S), Q304.3 (S)
- net HDRV1: now also Q301.4 (G)
- net HDRV2: now also Q303.4 (G)
- net LDRV1: now also Q302.4 (G)
- net LDRV2: now also Q304.4 (G)
- net SW1: now also Q301.1 (S), Q301.2 (S), Q301.3 (S), Q302.5 (D), Q302.6 (D), Q302.7 (D), Q302.8 (D)
- net SW2: now also Q303.1 (S), Q303.2 (S), Q303.3 (S), Q304.5 (D), Q304.6 (D), Q304.7 (D), Q304.8 (D)
- net SYS_24V: now also Q303.5 (D), Q303.6 (D), Q303.7 (D), Q303.8 (D)
- net VEH_DGATE: now also Q201.4 (G)
- net VEH_FET_MID: now also Q201.5 (D), Q201.6 (D), Q201.7 (D), Q201.8 (D), Q202.5 (D), Q202.6 (D), Q202.7 (D), Q202.8 (D)
- net VEH_FILTER: now also Q201.1 (S), Q201.2 (S), Q201.3 (S)
- net VEH_HGATE: now also Q202.4 (G)
- net VEH_PROT: now also Q202.1 (S), Q202.2 (S), Q202.3 (S), Q301.5 (D), Q301.6 (D), Q301.7 (D), Q301.8 (D)
Other:
- note added: "01: SINGLE 12 V INPUT"
- note added: "02: VEHICLE INPUT PROTECTION"
- note added: "03: LM5176 SINGLE-SOURCE BUCK-BOOST"
- note removed: "LM5176 SINGLE-SOURCE BUCK-BOOST"
- note removed: "LM5176 output directly supplies SYS_24V; no high-voltage source ORing is present."
- note removed: "SINGLE 12 V INPUT"
- note removed: "SYSTEM 24 V DISTRIBUTION"
- note removed: "SYS_24V has 264 uF converter output capacitance plus 19.547 uF distributed local bypass."
- note removed: "VEHICLE INPUT PROTECTION"
- company: ESP32-P4 Displayman Development Daughterboard -> sydude/ESP32-P4-Display-Development-Daughterboard
- title: Power -> ESP32-P4 Displayman Development Daughterboard
